Commit message: feature: add collision points to sesame robot

File: onshape/robot.urdf (robot description, URDF)
Before this commit: robot onshape, 9 links, 8 joints
Links:
- added link l3_p1, mass 1e-9
- added link l3_p2, mass 1e-9
- added link l3_p3, mass 1e-9
- added link l3_p4, mass 1e-9
- added link l4_p1, mass 1e-9
- added link l4_p2, mass 1e-9
- added link l4_p3, mass 1e-9
- added link l4_p4, mass 1e-9
- added link r3_p1, mass 1e-9
- added link r3_p2, mass 1e-9
- added link r3_p3, mass 1e-9
- added link r3_p4, mass 1e-9
- added link r4_p1, mass 1e-9
- added link r4_p2, mass 1e-9
- added link r4_p3, mass 1e-9
- added link r4_p4, mass 1e-9
Joints:
- added joint l3_p1_frame: type fixed, parent foot_joint_l3, child l3_p1, origin xyz=0.001905 0.04706 -0.0199857 rpy=-1.5708 1.5708 0, axis 0 0 0
- added joint l3_p2_frame: type fixed, parent foot_joint_l3, child l3_p2, origin xyz=0.001905 0.04706 -0.0120344 rpy=-1.5708 1.5708 0, axis 0 0 0
- added joint l3_p3_frame: type fixed, parent foot_joint_l3, child l3_p3, origin xyz=-0.00508 0.04706 -0.0199857 rpy=-1.5708 1.5708 0, axis 0 0 0
- added joint l3_p4_frame: type fixed, parent foot_joint_l3, child l3_p4, origin xyz=-0.00508 0.04706 -0.0123397 rpy=-1.5708 1.5708 0, axis 0 0 0
- added joint l4_p1_frame: type fixed, parent foot_joint_l4, child l4_p1, origin xyz=0.001905 -0.04706 -0.019813 rpy=1.5708 1.5708 0, axis 0 0 0
- added joint l4_p2_frame: type fixed, parent foot_joint_l4, child l4_p2, origin xyz=0.001905 -0.04706 -0.0120344 rpy=1.5708 1.5708 0, axis 0 0 0
- added joint l4_p3_frame: type fixed, parent foot_joint_l4, child l4_p3, origin xyz=-0.00508 -0.04706 -0.019813 rpy=1.5708 1.5708 0, axis 0 0 0
- added joint l4_p4_frame: type fixed, parent foot_joint_l4, child l4_p4, origin xyz=-0.00508 -0.04706 -0.0123397 rpy=1.5708 1.5708 0, axis 0 0 0
- added joint r3_p1_frame: type fixed, parent foot_joint_r3, child r3_p1, origin xyz=0.001905 -0.04706 -0.0195906 rpy=1.5708 1.5708 0, axis 0 0 0
- added joint r3_p2_frame: type fixed, parent foot_joint_r3, child r3_p2, origin xyz=0.001905 -0.04706 -0.0120344 rpy=1.5708 1.5708 0, axis 0 0 0
- added joint r3_p3_frame: type fixed, parent foot_joint_r3, child r3_p3, origin xyz=-0.00508 -0.04706 -0.0192853 rpy=1.5708 1.5708 0, axis 0 0 0
- added joint r3_p4_frame: type fixed, parent foot_joint_r3, child r3_p4, origin xyz=-0.00508 -0.04706 -0.0123397 rpy=1.5708 1.5708 0, axis 0 0 0
- added joint r4_p1_frame: type fixed, parent foot_joint_r4, child r4_p1, origin xyz=0.001905 0.04706 -0.0195906 rpy=-1.5708 1.5708 0, axis 0 0 0
- added joint r4_p2_frame: type fixed, parent foot_joint_r4, child r4_p2, origin xyz=0.001905 0.04706 -0.0120344 rpy=-1.5708 1.5708 0, axis 0 0 0
- added joint r4_p3_frame: type fixed, parent foot_joint_r4, child r4_p3, origin xyz=-0.00508 0.04706 -0.0192853 rpy=-1.5708 1.5708 0, axis 0 0 0
- added joint r4_p4_frame: type fixed, parent foot_joint_r4, child r4_p4, origin xyz=-0.00508 0.04706 -0.0123397 rpy=-1.5708 1.5708 0, axis 0 0 0

Commit message: feature: add full cad

File: onshape/robot.urdf (robot description, URDF)
Before this commit: robot onshape, 25 links, 24 joints
Links:
- link internal_frame: mass 0.058723 -> 0.0625592; geometry visual mesh filename=package://assets/bottom_cover.stl; visual mesh filename=package://assets/internal_frame.stl
