Commit message: feat: add base collision points

File: onshape/robot.urdf (robot description, URDF)
Before this commit: robot onshape, 25 links, 24 joints
Links:
- added link base_p1, mass 1e-9
- added link base_p2, mass 1e-9
- added link base_p3, mass 1e-9
- added link base_p4, mass 1e-9
Joints:
- added joint base_p1_frame: type fixed, parent internal_frame, child base_p1, origin xyz=-0.0371484 -0.0221984 -0.0161141 rpy=0 -0 0, axis 0 0 0
- added joint base_p2_frame: type fixed, parent internal_frame, child base_p2, origin xyz=-0.0371484 0.0126536 -0.0161141 rpy=0 -0 0, axis 0 0 0
- added joint base_p3_frame: type fixed, parent internal_frame, child base_p3, origin xyz=0.0349327 0.0126536 -0.0161141 rpy=0 -0 0, axis 0 0 0
- added joint base_p4_frame: type fixed, parent internal_frame, child base_p4, origin xyz=0.0349327 -0.0221984 -0.0161141 rpy=3.14159 -0 0, axis 0 0 0
